Commit message: update inertia, add ros2_control to urdf and udpate tricycle controller

File: rinkrover_description/description/robot.urdf.xacro (robot description, xacro)
@@ -4,3 +4,4 @@
     <xacro:include filename="materials.xacro"/>
     <xacro:include filename="robot_core.xacro"/>
+    <xacro:include filename="ros2_control.xacro"/>
 </robot>

File: rinkrover_description/description/robot_core.xacro (robot description, xacro)
@@ -2,4 +2,5 @@
 <robot xmlns:xacro="http://ros.org/wiki/xacro">
     <!---Based off Tricycle Controller and CarlikeBot example-->
+    <xacro:include filename="inertial_macros.xacro"/>
     <!--BASE LINK-->
     <link name="base_link" />
@@ -7,5 +8,5 @@
     <link name="chassis">
         <collision>
-        <origin xyz="${chassis_length/2} 0 ${chassis_height/2}"/>
+        <origin xyz="${(chassis_length/2)-0.45} 0 ${chassis_height/2}"/>
         <geometry>
             <box size="${chassis_length} ${chassis_width} ${chassis_height}"/>
@@ -19,9 +20,7 @@
             <material name="grey"/>
         </visual>
-        <!-- <inertial>
-        <origin xyz="0 0 0" rpy="0 0 0" />
-        <mass value="1" />
-        <inertia ixx="0.126164" ixy="0.0" ixz="0.0" iyy="0.416519" iyz="0.0" izz="0.481014" />
-        </inertial> -->
+        <xacro:inertial_box mass="1" x="${chassis_length}" y="${chassis_width}" z="${chassis_height}">
+            <origin xyz="${(chassis_length/2)-0.45} 0 ${chassis_height/2}"/>
+        </xacro:inertial_box>
     </link>
     <joint name="chassis_joint" type="fixed">
@@ -43,8 +42,7 @@
             <material name="black"/>
         </visual>
-        <!-- <inertial>
-        <mass value="2" />
-        <inertia ixx="0.145833" ixy="0.0" ixz="0.0" iyy="0.145833" iyz="0.0" izz="0.125" />
-        </inertial> -->
+        <xacro:inertial_cylinder mass="0.1" length="${wheel_width}" radius="${wheel_radius}">
+            <origin xyz="0 ${track_width/2} 0" rpy="-${pi/2} 0 0"/>
+        </xacro:inertial_cylinder>
     </link>
     <joint name="rear_left_wheel_joint" type="continuous">
@@ -68,8 +66,7 @@
             <material name="black"/>
         </visual>
-    <!-- <inertial>
-      <mass value="2" />
-      <inertia ixx="0.145833" ixy="0.0" ixz="0.0" iyy="0.145833" iyz="0.0" izz="0.125" />
-    </inertial> -->
+        <xacro:inertial_cylinder mass="0.1" length="${wheel_width}" radius="${wheel_radius}">
+            <origin xyz="0 -${track_width/2} 0" rpy="-${pi/2} 0 0"/>
+        </xacro:inertial_cylinder>
     </link>
     <joint name="rear_right_wheel_joint" type="continuous">
@@ -78,5 +75,4 @@
         <origin xyz="0 -${track_width/2} 0" rpy="-${pi/2} 0 0"/>
         <axis xyz="0 0 1"/>
-        <!-- <dynamics damping="0.2" /> -->
     </joint>
     <!-- FRONT Steering Link -->
@@ -128,4 +124,7 @@
         <material name="black"/>
         </visual>
+        <xacro:inertial_cylinder mass="0.1" length="${wheel_width}" radius="${wheel_radius}">
+            <origin xyz="${wheelbase/2} ${track_width/2} 0" rpy="-${pi/2} ${pi/2} 0"/>
+        </xacro:inertial_cylinder>
     </link>
     <joint name="front_right_wheel_joint" type="continuous">
@@ -149,4 +148,7 @@
         <material name="black"/>
         </visual>
+        <xacro:inertial_cylinder mass="0.1" length="${wheel_width}" radius="${wheel_radius}">
+            <origin xyz="${wheelbase/2} -${track_width/2} 0" rpy="-${pi/2} ${pi/2} 0"/>
+        </xacro:inertial_cylinder>
     </link>
     <joint name="front_left_wheel_joint" type="continuous">

Commit message: split real and sim xacros

File: rinkrover_description/description/robot.urdf.xacro (robot description, xacro)
@@ -4,4 +4,4 @@
     <xacro:include filename="materials.xacro"/>
     <xacro:include filename="robot_core.xacro"/>
-    <xacro:include filename="ros2_control.xacro"/>
+    <xacro:include filename="ros2_control_sim.xacro"/>
 </robot>

File: rinkrover_description/description/ros2_control.xacro (robot description, xacro)
@@ -1,8 +1,8 @@
 <?xml version="1.0"?>
-<robot xmlns:xacro="http://www.ros.org/wiki/xacro" >
-    <ros2_control name="GazeboSystem" type="system">
+<robot xmlns:xacro="http://www.ros.org/wiki/xacro">
+    <xacro:macro name="rinkrover_ros2_control">
+        <ros2_control name="RRSystem" type="system">
         <hardware>
-            <!-- Hardware Interface -->
-            <plugin>ign_ros2_control/IgnitionSystem</plugin>
+            <plugin>rinkrover_hardware/RRSystemHardware</plugin>
         </hardware>
         <joint name="steering_joint">
@@ -15,9 +15,5 @@
             <state_interface name="position"/>
         </joint>
-    </ros2_control>
-    <gazebo>
-        <plugin filename="libign_ros2_control-system.so" name="ign_ros2_control::IgnitionROS2ControlPlugin">
-            <parameters>$(find rinkrover_description)/config/tricycle_drive_controller.yaml</parameters>
-        </plugin>
-    </gazebo>
+        </ros2_control>
+    </xacro:macro>
 </robot>
