Commit message: fix encoder reading and joint state callback

File: rinkrover_description/description/robot_properties.xacro (robot description, xacro)
@@ -2,5 +2,5 @@
 <robot xmlns:xacro="http://www.ros.org/wiki/xacro">
     <!-- Define basic properties -->
-    <xacro:property name="wheel_radius" value="0.125"/>
+    <xacro:property name="wheel_radius" value="0.127"/>
     <xacro:property name="wheel_width" value="0.09"/>
     <xacro:property name="chassis_length" value="1.691"/>
