Commit message: get gazebo simulation working

File: rinkrover_description/description/robot_core.xacro (robot description, xacro)
@@ -18,7 +18,7 @@
                 <box size="${chassis_length} ${chassis_width} ${chassis_height}"/>
             </geometry>
-            <material name="grey"/>
+            <material name="blue"/>
         </visual>
-        <xacro:inertial_box mass="1" x="${chassis_length}" y="${chassis_width}" z="${chassis_height}">
+        <xacro:inertial_box mass="0.05" x="${chassis_length}" y="${chassis_width}" z="${chassis_height}">
             <origin xyz="${(chassis_length/2)-0.45} 0 ${chassis_height/2}"/>
         </xacro:inertial_box>
@@ -29,4 +29,7 @@
         <origin xyz="-0.45 0 0"/>
     </joint>
+    <gazebo reference="chassis">
+        <material>Gazebo/Blue</material>
+    </gazebo>
     <!-- BACK left wheel Link -->
     <link name="rear_left_wheel">
@@ -42,5 +45,5 @@
             <material name="black"/>
         </visual>
-        <xacro:inertial_cylinder mass="0.1" length="${wheel_width}" radius="${wheel_radius}">
+        <xacro:inertial_cylinder mass="5" length="${wheel_width}" radius="${wheel_radius}">
             <origin xyz="0 ${track_width/2} 0" rpy="-${pi/2} 0 0"/>
         </xacro:inertial_cylinder>
@@ -53,4 +56,7 @@
         <!-- <dynamics damping="0.2" /> -->
     </joint>
+    <gazebo reference="rear_left_wheel">
+        <material>Gazebo/Black</material>
+    </gazebo>
     <!-- BACK right wheel Link -->
     <link name="rear_right_wheel">
@@ -66,5 +72,5 @@
             <material name="black"/>
         </visual>
-        <xacro:inertial_cylinder mass="0.1" length="${wheel_width}" radius="${wheel_radius}">
+        <xacro:inertial_cylinder mass="5" length="${wheel_width}" radius="${wheel_radius}">
             <origin xyz="0 -${track_width/2} 0" rpy="-${pi/2} 0 0"/>
         </xacro:inertial_cylinder>
@@ -76,4 +82,7 @@
         <axis xyz="0 0 1"/>
     </joint>
+    <gazebo reference="rear_right_wheel">
+        <material>Gazebo/Black</material>
+    </gazebo>
     <!-- FRONT Steering Link -->
     <link name="steering_link">
@@ -84,4 +93,7 @@
         <material name="black" />
         </visual>
+        <xacro:inertial_box mass="0.001" x="0.01" y="0.01" z="0.01">
+            <origin xyz="0 0 0"/>
+        </xacro:inertial_box>
     </link>
     <joint name="steering_joint" type="continuous">
@@ -100,8 +112,11 @@
         </visual>
         <collision>
-        <geometry>
-            <cylinder radius="${wheel_radius}" length="${wheel_width}"/>
-        </geometry>
+            <geometry>
+                <cylinder radius="${wheel_radius}" length="${wheel_width}"/>
+            </geometry>
         </collision>
+        <xacro:inertial_cylinder mass="10" length="${wheel_width}" radius="${wheel_radius}">
+            <origin xyz="0 0 0" rpy="-${pi/2} ${pi/2} 0"/>
+        </xacro:inertial_cylinder>
     </link>
     <joint name="virtual_traction_joint" type="continuous">
@@ -113,9 +128,9 @@
     <!-- Front Right Wheel-->
     <link name="front_right_wheel">
-        <collision>
+        <!-- <collision>
             <geometry>
             <cylinder length="${wheel_width}" radius="${wheel_radius}"/>
             </geometry>
-        </collision>
+        </collision> -->
         <visual>
             <geometry>
@@ -124,5 +139,5 @@
         <material name="black"/>
         </visual>
-        <xacro:inertial_cylinder mass="0.1" length="${wheel_width}" radius="${wheel_radius}">
+        <xacro:inertial_cylinder mass="0.01" length="${wheel_width}" radius="${wheel_radius}">
             <origin xyz="${wheelbase/2} ${track_width/2} 0" rpy="-${pi/2} ${pi/2} 0"/>
         </xacro:inertial_cylinder>
@@ -135,11 +150,14 @@
         <mimic joint="virtual_traction_joint" multiplier="1.0" offset="0.0"/>
     </joint>
+    <gazebo reference="front_right_wheel">
+        <material>Gazebo/Black</material>
+    </gazebo>
     <!-- Front Left Wheel-->
     <link name="front_left_wheel">
-        <collision>
+        <!-- <collision>
             <geometry>
             <cylinder length="${wheel_width}" radius="${wheel_radius}"/>
             </geometry>
-        </collision>
+        </collision> -->
         <visual>
             <geometry>
@@ -148,5 +166,5 @@
         <material name="black"/>
         </visual>
-        <xacro:inertial_cylinder mass="0.1" length="${wheel_width}" radius="${wheel_radius}">
+        <xacro:inertial_cylinder mass="0.01" length="${wheel_width}" radius="${wheel_radius}">
             <origin xyz="${wheelbase/2} -${track_width/2} 0" rpy="-${pi/2} ${pi/2} 0"/>
         </xacro:inertial_cylinder>
@@ -159,22 +177,6 @@
         <mimic joint="virtual_traction_joint" multiplier="1.0" offset="0.0"/>
     </joint>
-  <!-- <ros2_control name="GazeboSystem" type="system">
-    <hardware>
-      <plugin>gazebo_ros2_control/GazeboSystem</plugin>
-    </hardware>
-    <joint name="steering_joint">
-      <command_interface name="position" />
-      <state_interface name="position" />
-    </joint>
-    <joint name="traction_joint">
-      <command_interface name="velocity" />
-      <state_interface name="velocity" />
-      <state_interface name="position" />
-    </joint>
-  </ros2_control>
-  <gazebo>
-    <plugin filename="libgazebo_ros2_control.so" name="gazebo_ros2_control">
-      <parameters>$(find gazebo_ros2_control_demos)/config/tricycle_drive_controller.yaml</parameters>
-    </plugin>
-  </gazebo> -->
+    <gazebo reference="front_left_wheel">
+        <material>Gazebo/Black</material>
+    </gazebo>
 </robot>

File: rinkrover_description/description/ros2_control.xacro (robot description, xacro)
@@ -4,19 +4,12 @@
         <hardware>
             <!-- Hardware Interface -->
-            <plugin>gz_ros2_control/GazeboSimSystem</plugin>
+            <plugin>ign_ros2_control/IgnitionSystem</plugin>
         </hardware>
         <joint name="steering_joint">
-            <command_interface name="velocity">
-                <param name="min">-10</param>
-                <param name="max">10</param>
-            </command_interface>
-            <state_interface name="velocity"/>
+            <command_interface name="position"/>
             <state_interface name="position"/>
         </joint>
         <joint name="virtual_traction_joint">
-            <command_interface name="velocity">
-                <param name="min">-10</param>
-                <param name="max">10</param>
-            </command_interface>
+            <command_interface name="velocity"/>
             <state_interface name="velocity"/>
             <state_interface name="position"/>
@@ -24,6 +17,6 @@
     </ros2_control>
     <gazebo>
-        <plugin filename="gz_ros2_control-system" name="gz_ros2_control::GazeboSimROS2ControlPlugin">
-        <parameters>$(find rinkrover_description)/config/tricycle_drive_controller.yaml</parameters>
+        <plugin filename="libign_ros2_control-system.so" name="ign_ros2_control::IgnitionROS2ControlPlugin">
+            <parameters>$(find rinkrover_description)/config/tricycle_drive_controller.yaml</parameters>
         </plugin>
     </gazebo>

Commit message: get LIDAR working with gazebo sim

File: rinkrover_description/description/robot_core.xacro (robot description, xacro)
@@ -164,5 +164,5 @@
             <cylinder length="${wheel_width}" radius="${wheel_radius}"/>
             </geometry>
-        <material name="black"/>
+            <material name="black"/>
         </visual>
         <xacro:inertial_cylinder mass="0.01" length="${wheel_width}" radius="${wheel_radius}">
@@ -180,3 +180,56 @@
         <material>Gazebo/Black</material>
     </gazebo>
+    <!--LIDAR LINK-->
+    <link name="base_scan">
+        <xacro:inertial_cylinder mass="0.01" length="${wheel_width}" radius="${wheel_radius}">
+            <origin xyz="${wheelbase/2} 0 ${chassis_height}" rpy="0 0 0" />
+        </xacro:inertial_cylinder>
+        <visual name="lidar_sensor_visual">
+            <geometry>
+                <cylinder length="${wheel_width}" radius="${wheel_radius}"/>
+            </geometry>
+        </visual>
+    </link>
+    <gazebo reference="base_scan">
+    <sensor name="lidar_sensor" type="gpu_lidar">
+        <pose relative_to='base_scan'>0 0 0 0 0 0</pose>
+        <always_on>1</always_on>
+        <visualize>true</visualize>
+        <update_rate>10</update_rate>
+        <topic>scan</topic>
+        <ignition_frame_id>base_scan</ignition_frame_id>
+        <ray>
+          <scan>
+            <horizontal>
+              <samples>360</samples>
+              <resolution>1.000000</resolution>
+              <min_angle>0.000000</min_angle>
+              <max_angle>6.280000</max_angle>
+            </horizontal>
+          </scan>
+          <range>
+            <min>0.120000</min>
+            <max>12.0</max>
+            <resolution>0.015000</resolution>
+          </range>
+          <noise>
+            <type>gaussian</type>
+            <mean>0.0</mean>
+            <stddev>0.01</stddev>
+          </noise>
+        </ray>
+      </sensor>
+    </gazebo>
+    <gazebo>
+            <plugin
+        filename="libignition-gazebo6-sensors-system.so"
+        name="ignition::gazebo::systems::Sensors">
+        <render_engine>ogre2</render_engine>
+        </plugin>
+    </gazebo>
+    <joint name="lidar_joint" type="fixed">
+        <parent link="base_link" />
+        <child link="base_scan" />
+        <origin xyz="${wheelbase/2} 0 ${chassis_height + 0.2}" rpy="0 0 0" />
+    </joint>
 </robot>

Commit message: get SLAM mapping working and add first pass sim map

File: rinkrover_description/description/robot_core.xacro (robot description, xacro)
@@ -5,4 +5,12 @@
     <!--BASE LINK-->
     <link name="base_link" />
+    <!--BASE FOOTPRINT LINK-->
+    <joint name="base_footprint_joint" type="fixed">
+        <parent link="base_link" />
+        <child link="base_footprint" />
+        <origin xyz="0 0 0" rpy="0 0 0"/>
+    </joint>
+    <link name="base_footprint">
+    </link>
     <!-- CHASSIS LINK-->
     <link name="chassis">
@@ -231,5 +239,5 @@
         <parent link="base_link" />
         <child link="base_scan" />
-        <origin xyz="${wheelbase/2} 0 ${chassis_height + 0.2}" rpy="0 0 0" />
+        <origin xyz="${wheelbase/2} 0 ${chassis_height + wheel_width/2}" rpy="0 0 0" />
     </joint>
 </robot>

Commit message: minor controller tuning

File: rinkrover_description/description/robot_core.xacro (robot description, xacro)
@@ -97,7 +97,7 @@
         <visual>
         <geometry>
-            <box size="0.01 0.01 0.01" />
-        </geometry>
-        <material name="black" />
+            <box size="0.1 0.1 0.1" />
+        </geometry>
+        <material name="orange" />
         </visual>
         <xacro:inertial_box mass="0.001" x="0.01" y="0.01" z="0.01">
@@ -105,10 +105,14 @@
         </xacro:inertial_box>
     </link>
-    <joint name="steering_joint" type="continuous">
+    <joint name="steering_joint" type="revolute">
         <origin xyz="${wheelbase} 0 0" rpy="0 0 0" />
         <parent link="chassis" />
         <child link="steering_link" />
         <axis xyz="0 0 1" />
-    </joint>
+        <limit effort="5.0" velocity="2.0" lower="-0.78" upper="0.78"/>
+    </joint>
+        <gazebo reference="steering_link">
+        <material>Gazebo/Black</material>
+    </gazebo>
     <!-- VIRTUAL traction wheel link -->
     <link name="virtual_traction_link">
@@ -117,5 +121,5 @@
             <cylinder radius="${wheel_radius}" length="${wheel_width}"/>
         </geometry>
-        <material name="invisible" />
+        <material name="white" />
         </visual>
         <collision>
@@ -147,7 +151,4 @@
         <material name="black"/>
         </visual>
-        <xacro:inertial_cylinder mass="0.01" length="${wheel_width}" radius="${wheel_radius}">
-            <origin xyz="${wheelbase/2} ${track_width/2} 0" rpy="-${pi/2} ${pi/2} 0"/>
-        </xacro:inertial_cylinder>
     </link>
     <joint name="front_right_wheel_joint" type="continuous">
@@ -174,7 +175,4 @@
             <material name="black"/>
         </visual>
-        <xacro:inertial_cylinder mass="0.01" length="${wheel_width}" radius="${wheel_radius}">
-            <origin xyz="${wheelbase/2} -${track_width/2} 0" rpy="-${pi/2} ${pi/2} 0"/>
-        </xacro:inertial_cylinder>
     </link>
     <joint name="front_left_wheel_joint" type="continuous">

Commit message: fix encoder reading, update xacro with better measurements, get lidar running

File: rinkrover_description/description/robot_core.xacro (robot description, xacro)
@@ -16,5 +16,5 @@
     <link name="chassis">
         <collision>
-        <origin xyz="${(chassis_length/2)-0.45} 0 ${chassis_height/2}"/>
+        <origin xyz="${(chassis_length/2)} 0 ${chassis_height/2}"/>
         <geometry>
             <box size="${chassis_length} ${chassis_width} ${chassis_height}"/>
@@ -22,5 +22,5 @@
         </collision>
         <visual>
-            <origin xyz="${(chassis_length/2)-0.45} 0 ${chassis_height/2}"/>
+            <origin xyz="${(chassis_length/2)} 0 ${chassis_height/2}"/>
             <geometry>
                 <box size="${chassis_length} ${chassis_width} ${chassis_height}"/>
@@ -29,5 +29,5 @@
         </visual>
         <xacro:inertial_box mass="0.05" x="${chassis_length}" y="${chassis_width}" z="${chassis_height}">
-            <origin xyz="${(chassis_length/2)-0.45} 0 ${chassis_height/2}"/>
+            <origin xyz="${(chassis_length/2)} 0 ${chassis_height/2}"/>
         </xacro:inertial_box>
     </link>
@@ -35,5 +35,5 @@
         <parent link="base_link" />
         <child link="chassis" />
-        <origin xyz="-0.45 0 0"/>
+        <origin xyz="-${wheel_radius+0.45} 0 0"/>
     </joint>
     <gazebo reference="chassis">
@@ -107,5 +107,5 @@
     <joint name="steering_joint" type="revolute">
         <origin xyz="${wheelbase} 0 0" rpy="0 0 0" />
-        <parent link="chassis" />
+        <parent link="base_link" />
         <child link="steering_link" />
         <axis xyz="0 0 1" />
@@ -155,5 +155,5 @@
         <parent link="base_link" />
         <child link="front_right_wheel" />
-        <origin xyz="${wheelbase/2} ${track_width/2} 0" rpy="-${pi/2} ${pi/2} 0"/>
+        <origin xyz="${wheelbase} ${track_width/2} 0" rpy="-${pi/2} ${pi/2} 0"/>
         <axis xyz="0 0 1"/>
         <mimic joint="virtual_traction_joint" multiplier="1.0" offset="0.0"/>
@@ -179,5 +179,5 @@
         <parent link="base_link" />
         <child link="front_left_wheel" />
-        <origin xyz="${wheelbase/2} -${track_width/2} 0" rpy="-${pi/2} ${pi/2} 0"/>
+        <origin xyz="${wheelbase} -${track_width/2} 0" rpy="-${pi/2} ${pi/2} 0"/>
         <axis xyz="0 0 1"/>
         <mimic joint="virtual_traction_joint" multiplier="1.0" offset="0.0"/>
@@ -237,5 +237,5 @@
         <parent link="base_link" />
         <child link="base_scan" />
-        <origin xyz="${wheelbase/2} 0 ${chassis_height + wheel_width/2}" rpy="0 0 0" />
+        <origin xyz="${wheelbase/2} 0 ${chassis_height + wheel_width/2}" rpy="0 0 -3.14159" />
     </joint>
 </robot>

Commit message: publish IMU data on IMU topic

File: rinkrover_description/description/robot_core.xacro (robot description, xacro)
@@ -239,3 +239,27 @@
         <origin xyz="${wheelbase/2} 0 ${chassis_height + wheel_width/2}" rpy="0 0 -3.14159" />
     </joint>
+<!--IMU LINK-->
+    <link name="imu_link">
+        <origin xyz="0 0 0" rpy="0 0 0" />
+        <visual>
+            <origin xyz="0 0 0"/>
+            <geometry>
+                <box size="0.05 0.05 0.05"/>
+            </geometry>
+            <material name="blue"/>
+        </visual>
+    </link>
+    <gazebo reference="imu_link">
+        <sensor name="imu_sensor" type="imu">
+            <pose relative_to='base_scan'>0 0 0 0 0 0</pose>
+            <parent link="imu_link"/>
+            <topic name="imu_data" />
+            <update_rate>10</update_rate>
+        </sensor>
+    </gazebo>
+    <joint name="imu_joint" type="fixed">
+        <parent link="base_link"/>
+        <child link="imu_link"/>
+        <origin xyz="0 0 0" rpy="0 0 0"/>
+    </joint>
 </robot>

File: rinkrover_description/description/ros2_control.xacro (robot description, xacro)
@@ -23,4 +23,16 @@
         <state_interface name="position"/>
     </joint>
+    <sensor name="imu_sensor" type="imu_sensor">
+        <state_interface name="orientation.w"/>
+        <state_interface name="orientation.x"/>
+        <state_interface name="orientation.y"/>
+        <state_interface name="orientation.z"/>
+        <state_interface name="angular_velocity.x"/>
+        <state_interface name="angular_velocity.y"/>
+        <state_interface name="angular_velocity.z"/>
+        <state_interface name="linear_acceleration.x"/>
+        <state_interface name="linear_acceleration.y"/>
+        <state_interface name="linear_acceleration.z"/>
+    </sensor>
     </ros2_control>
 </robot>

Commit message: update EKF params and enable for hardware testing

File: rinkrover_description/description/robot_core.xacro (robot description, xacro)
@@ -189,5 +189,5 @@
     <link name="base_scan">
         <xacro:inertial_cylinder mass="0.01" length="${wheel_width}" radius="${wheel_radius}">
-            <origin xyz="${wheelbase/2} 0 ${chassis_height}" rpy="0 0 0" />
+            <origin xyz="${wheelbase/2} 0 0" rpy="0 0 0" />
         </xacro:inertial_cylinder>
         <visual name="lidar_sensor_visual">
@@ -237,5 +237,5 @@
         <parent link="base_link" />
         <child link="base_scan" />
-        <origin xyz="${wheelbase/2} 0 ${chassis_height + wheel_width/2}" rpy="0 0 -3.14159" />
+        <origin xyz="${wheelbase/2} 0 0.5" rpy="0 0 -3.14159" />
     </joint>
 <!--IMU LINK-->
